File: hardware/trichter/power.kicad_sch (KiCad schematic)
At the start: 19 parts, among them J6 USB_C_Receptacle, J8 Conn_01x03_Pin, J9 Conn_01x02_Pin, SW2 SW_DIP_x01, U2 AP7361C-33E

Commit message: Layout & Routing.
Parts:
- removed J6: USB_C_Receptacle, symbol Connector:USB_C_Receptacle
- removed SW2: SW_DIP_x01, symbol Switch:SW_DIP_x01
- added J6: USB4110-GF-A, USB4110-GF-A_GCT, symbol morb:USB4110-GF-A
- added SW2: SW_SPDT, morb:SW_SPDT_ANT11SF1CQE, symbol Switch:SW_SPDT
- C4, C5: footprint (none) -> Capacitor_SMD:C_0805_2012Metric_Pad1.18x1.45mm_HandSolder
- D2: footprint (none) -> LED_SMD:LED_0603_1608Metric_Pad1.05x0.95mm_HandSolder; Part Number (none) -> LTST-C190GKT
- J8: footprint (none) -> Connector_PinHeader_2.54mm:PinHeader_1x03_P2.54mm_Vertical
- J9: footprint (none) -> Connector_PinHeader_2.54mm:PinHeader_1x02_P2.54mm_Vertical
- R1, R4, R6: footprint (none) -> Resistor_SMD:R_0805_2012Metric_Pad1.20x1.40mm_HandSolder
- TP1, TP2, TP3, TP4, TP5, TP6, TP7, TP8: footprint (none) -> TestPoint:TestPoint_THTPad_D1.5mm_Drill0.7mm
Connections:
- net +5V: now also SW2.1 (A)
- net GND: now also J6.15 (SHIELD), J6.16 (SHIELD), J6.17 (SHIELD), J6.18 (SHIELD), J6.A1-B12 (GND), J6.A12-B1 (GND)
- net VBUS: now also J6.A4-B9 (VBUS), J6.A9-B4 (VBUS)
- net at J8.2 (Pin_2): now also SW2.2 (B)
- net at R6.1: now also J6.B5 (CC2)
- net at R1.1: now also J6.A5 (CC1)
- new net D_N: J6.A7 (DN1), J6.B7 (DN2)
- new net D_P: J6.A6 (DP1), J6.B6 (DP2)
- no-connect marks 14 -> 3
Other:
- moved on the sheet: D2, R1, R4, R6, TP8

Commit message: Export gerber files and add BOM.
Parts:
- R4: value 10k -> 390
Changed lines of the file:
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@@
     (stroke (width 0) (type default))
   )
-  (text_box "Resistor value depends on which LED will be used"
-    (at 162.56 76.2 0) (size 20.32 7.62)
+  (text_box "See D1 for resistor calculation"
+    (at 161.29 85.09 0) (size 12.7 7.62)
     (stroke (width 0) (type default))
     (fill (type none))
@@
       (effects (font (size 1.27 1.27)) (justify left))
     )
-    (property "Value" "10k" (at 153.67 90.17 0)
+    (property "Value" "390" (at 153.67 90.17 0)
       (effects (font (size 1.27 1.27)) (justify left))
     )
