File: hardware/trichter/trichter.kicad_pcb (KiCad board)
At the start: 2 copper layers, 64.9 x 35 mm, 38 parts, among them J1 Conn_01x03_Pin, J2 Conn_01x09_Pin, J3 Conn_01x04_Pin, J4 Conn_01x04_Pin, J5 Conn_02x06_Pin, J6 USB4110-GF-A, J7 Connector Flow Sensor, J8 Conn_01x03_Pin, J9 Conn_01x02_Pin, SW1 SW_Push, SW2 SW_SPDT, U1 STM32C051K8T6, U2 AP7361C-33E

Commit message: Export gerber files and add BOM.
Routing:
- net GND: track 12.4 -> 14.4 mm, vias 81 -> 93
