File: hardware/trichter/trichter.kicad_sch (KiCad schematic)
At the start: 5 parts, among them J7 Connector Flow Sensor

Commit message: Layout & Routing.
Parts:
- C6: footprint (none) -> Capacitor_SMD:C_0603_1608Metric_Pad1.08x0.95mm_HandSolder
- C7: footprint (none) -> Capacitor_SMD:C_0805_2012Metric_Pad1.18x1.45mm_HandSolder
- D1: footprint (none) -> LED_SMD:LED_0603_1608Metric_Pad1.05x0.95mm_HandSolder; Part Number (none) -> LTST-C190GKT
- R3: footprint (none) -> Resistor_SMD:R_0805_2012Metric_Pad1.20x1.40mm_HandSolder
Changed lines of the file:
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@@
       (effects (font (size 1.27 1.27)) (justify right))
     )
-    (property "Footprint" "" (at 168.91 49.53 0)
+    (property "Footprint" "LED_SMD:LED_0603_1608Metric_Pad1.05x0.95mm_HandSolder" (at 168.91 49.53 0)
       (effects (font (size 1.27 1.27)) hide)
     )
@@
       (effects (font (size 1.27 1.27)) hide)
     )
+    (property "Part Number" "LTST-C190GKT" (at 168.91 49.53 90)
+      (effects (font (size 1.27 1.27)) hide)
+    )
     (pin "2")
     (pin "1")
@@
       (effects (font (size 1.27 1.27)) (justify left))
     )
-    (property "Footprint" "" (at 182.5752 34.29 0)
+    (property "Footprint" "Capacitor_SMD:C_0603_1608Metric_Pad1.08x0.95mm_HandSolder" (at 182.5752 34.29 0)
       (effects (font (size 1.27 1.27)) hide)
     )
@@
       (effects (font (size 1.27 1.27)) (justify left))
     )
-    (property "Footprint" "" (at 167.132 59.69 90)
+    (property "Footprint" "Resistor_SMD:R_0805_2012Metric_Pad1.20x1.40mm_HandSolder" (at 167.132 59.69 90)
       (effects (font (size 1.27 1.27)) hide)
     )
@@
       (effects (font (size 1.27 1.27)) (justify left))
     )
-    (property "Footprint" "" (at 169.8752 34.29 0)
-      (effects (font (size 1.27 1.27)) hide)
-    )
+    (property "Footprint" "Capacitor_SMD:C_0805_2012Metric_Pad1.18x1.45mm_HandSolder" (at 169.8752 34.29 0)
+      (effects (font (size 1.27 1.27)) hide)
+    )

Commit message: Export gerber files and add BOM.
Parts:
- R3: value 1k -> 390
Changed lines of the file:
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@@
     (stroke (width 0) (type default))
   )
-  (text_box "Resistor value depends on which LED will be used"
-    (at 143.51 55.88 0) (size 20.32 7.62)
+  (text_box "- Flow sensor outputs >4.7V @ max. 10mA\n- LED is 5mA @ 2.75V\n-> 1.95V over R\n-> R = 1.95V / 5mA = 390 Ohm"
+    (at 176.53 57.15 0) (size 45.72 10.16)
     (stroke (width 0) (type default))
     (fill (type none))
@@
       (effects (font (size 1.27 1.27)) (justify left))
     )
-    (property "Value" "1k" (at 171.45 60.96 0)
-      (effects (font (size 1.27 1.27)) (justify left))
-    )
+    (property "Value" "390" (at 171.45 60.96 0)
+      (effects (font (size 1.27 1.27)) (justify left))
+    )
